File: proj1-led-torch/proj1-led-torch.kicad_sch (KiCad schematic)
At the start: 4 parts, among them SW1 SW_DPST_x2

Commit message: finished LED Torch
Changed lines of the file:
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@@
 		(on_board yes)
 		(dnp no)
-		(fields_autoplaced yes)
 		(property "Reference" "SW1"
 			(at 130.81 69.85 0)
@@
 		)
 		(property "Footprint" "Button_Switch_THT:SW_TH_Tactile_Omron_B3F-10xx"
-			(at 130.81 76.2 0)
+			(at 133.096 67.31 0)
 			(effects
 				(font
-					(size 1.27 1.27)
+					(size 0.5 0.5)
 				)
-				(hide yes)
 			)
 		)

Commit message: added files
Parts:
- added U1: ~, Package_DIP:DIP-8_W7.62mm_Socket_LongPads, symbol mikes-lib:NA555_MG
Changed lines of the file:
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@@
+	)
+	(symbol
+		(lib_id "mikes-lib:NA555_MG")
+		(at 173.99 80.01 0)
+		(unit 1)
+		(exclude_from_sim no)
+		(in_bom yes)
+		(on_board yes)
+		(dnp no)
+		(property "Reference" "U1"
+			(at 175.26 69.85 0)
+			(effects
+				(font
+					(size 1.27 1.27)
+				)
+				(justify left)
+			)
+		)
+		(property "Value" "~"
+			(at 176.1841 67.31 0)
+			(effects
+				(font
+					(size 1.27 1.27)
+				)
+				(justify left)
+			)
+		)
+		(property "Footprint" "Package_DIP:DIP-8_W7.62mm_Socket_LongPads"
+			(at 173.99 80.01 0)
+			(effects
+				(font
+					(size 1.27 1.27)
+				)
+				(hide yes)
+			)
+		)
+		(property "Datasheet" ""
+			(at 173.99 80.01 0)
+			(effects
+				(font
+					(size 1.27 1.27)
+				)
+				(hide yes)
+			)
+		)
+		(property "Description" "Mike's NA555 Symbol"
+			(at 173.99 80.01 0)
+			(effects
+				(font
+					(size 1.27 1.27)
+				)
+				(hide yes)
+			)
+		)
+		(pin "4"
+		)
+		(pin "5"
+		)
+		(pin "6"
+		)
+		(pin "8"
+		)
+		(pin "3"
+		)
+		(pin "7"
+		)
+		(pin "1"
+		)
+		(pin "2"
+		)
+		(instances
+			(project "proj1-led-torch"
+				(path "/f379e36e-d683-400b-afca-915f9d02195f"
+					(reference "U1")
+					(unit 1)
+				)
+			)
+		)
 	)
 	(symbol
