File: breadboard-power-supply/breadboard-power-supply.kicad_sch (KiCad schematic)
At the start: 17 parts, among them J1 Conn_01x02_Pin, J2 Conn_01x02_Pin, J3 Conn_01x03_Pin, J4 Conn_01x03_Pin, J5 Screw_Terminal_01x02, J6 Barrel_Jack_Switch, J7 Screw_Terminal_01x02, SW1 EG1218, U1 LM7805_TO220, U2 LM317_TO-220

Commit message: added breadboard power supply project
Parts:
- D1: Purpose (none) -> Power input indicator
- J1, J2: Purpose (none) -> Output to breadboard
- J3: Purpose (none) -> Output voltage selector 2
- J4: Purpose (none) -> Output voltage selector 1
- J5, J7: Purpose (none) -> Output to jumper wires
- SW1: footprint SW_1218_EWI -> Button_Switch_THT:SW_Slide-03_Wuerth-WS-SLTV_10x2.5x6.4_P2.54mm
Connections:
- net PWR_output renamed PWR_OUT_BOTTOM
Other:
- note added: "3.3V Circuit"
- note added: "I flipped screw terminals so that pin 1 is GND"
- note added: "Input and 5V ciruit"
- note added: "Output and Switches"
