File: mcu-datalogger/mcu-datalogger.kicad_sch (KiCad schematic)
At the start: 25 parts, among them U1 24LC1025, U2 24LC1025, U3 DS1337S_, U4 ATMEGA328P-AU, Y1 Crystal, Y2 Crystal

Commit message: updated symbol values
Parts:
- C1, C4: value C -> 0.1uF
- C2, C3: value C -> 22pF
- C5: value C_Polarized -> 100nF
- R1, R6: value R -> 4.7k
- R2, R3, R7: value R -> 10K
- R4, R5: value R -> 330
- Y1: value Crystal -> 16MHz
- Y2: value Crystal -> 32.768 KHz
Other:
- moved on the sheet: BT1
Changed lines of the file:
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@@
 			)
 		)
-		(property "Value" "R"
+		(property "Value" "10K"
 			(at 189.23 104.14 90)
 			(effects
@@
 			)
 		)
-		(property "Value" "Crystal"
+		(property "Value" "32.768 KHz"
 			(at 34.29 72.39 0)
 			(effects
@@
 			)
 		)
+		(property "Purpose" ""
+			(at 34.29 77.47 0)
+			(effects
+				(font
+					(size 1.27 1.27)
+				)
+			)
+		)
 		(pin "1"
 		)
@@
 			)
 		)
-		(property "Value" "C"
+		(property "Value" "0.1uF"
 			(at 175.26 45.72 90)
 			(effects
@@
 			)
 		)
-		(property "Value" "Crystal"
+		(property "Value" "16MHz"
 			(at 191.77 87.6299 90)
 			(effects
@@
 			)
 		)
-		(property "Value" "C"
+		(property "Value" "22pF"
 			(at 172.72 81.2799 0)
 			(effects
@@
 			)
 		)
-		(property "Value" "C_Polarized"
+		(property "Value" "100nF"
 			(at 251.46 65.1509 0)
 			(effects
@@
 			)
 		)
-		(property "Value" "R"
+		(property "Value" "330"
 			(at 167.64 67.31 90)
 			(effects
@@
 			)
 		)
-		(property "Value" "R"
+		(property "Value" "330"
 			(at 257.81 100.3299 0)
 			(effects
@@
 	(symbol
 		(lib_id "Device:Battery")
-		(at 256.54 63.5 0)
+		(at 264.16 63.5 0)
 		(unit 1)
 		(exclude_from_sim no)
@@
 		(fields_autoplaced yes)
 		(property "Reference" "BT1"
-			(at 260.35 61.6584 0)
+			(at 267.97 61.6584 0)
 			(effects
 				(font
@@
 		)
 		(property "Value" "Battery"
-			(at 260.35 64.1984 0)
-			(effects
-				(font
-					(size 1.27 1.27)
-				)
-				(justify left)
-			)
-		)
-		(property "Footprint" ""
-			(at 256.54 61.976 90)
+			(at 267.97 64.1984 0)
+			(effects
+				(font
+					(size 1.27 1.27)
+				)
+				(justify left)
+			)
+		)
+		(property "Footprint" ""
+			(at 264.16 61.976 90)
 			(effects
 				(font
@@
 		)
 		(property "Datasheet" "~"
-			(at 256.54 61.976 90)
+			(at 264.16 61.976 90)
 			(effects
 				(font
@@
 		)
 		(property "Description" "Multiple-cell battery"
-			(at 256.54 63.5 0)
+			(at 264.16 63.5 0)
 			(effects
 				(font
@@
 			)
 		)
-		(property "Value" "R"
+		(property "Value" "4.7k"
 			(at 128.27 165.0999 0)
 			(effects
@@
 			)
 		)
-		(property "Value" "C"
+		(property "Value" "22pF"
 			(at 172.72 93.9799 0)
 			(effects
@@
 			)
 		)
-		(property "Value" "R"
+		(property "Value" "4.7k"
 			(at 138.43 165.0999 0)
 			(effects
@@
 			)
 		)
-		(property "Value" "R"
+		(property "Value" "10K"
 			(at 114.3 76.1999 0)
 			(effects
@@
 			)
 		)
-		(property "Value" "C"
+		(property "Value" "0.1uF"
 			(at 130.81 76.1999 0)
 			(effects
@@
 			)
 		)
-		(property "Value" "R"
+		(property "Value" "10K"
 			(at 101.6 76.1999 0)
 			(effects

Commit message: associated footprints with symbols
Parts:
- BT1: footprint (none) -> Connector_PinHeader_2.54mm:PinHeader_1x02_P2.54mm_Vertical
- C1, C2, C3, C4, C5: footprint (none) -> Capacitor_SMD:C_0805_2012Metric
- D1, D2: footprint (none) -> LED_SMD:LED_0805_2012Metric
- H1, H2, H3, H4: footprint (none) -> MountingHole:MountingHole_2.1mm
- R1, R2, R3, R4, R5, R6, R7: footprint (none) -> Resistor_SMD:R_0805_2012Metric
- U1, U2: footprint (none) -> Package_SO:SOIC-8_5.23x5.23mm_P1.27mm
- Y1, Y2: footprint (none) -> Crystal:Crystal_SMD_5032-2Pin_5.0x3.2mm_HandSoldering
Changed lines of the file:
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@@
 			)
 		)
-		(property "Footprint" ""
+		(property "Footprint" "MountingHole:MountingHole_2.1mm"
 			(at 185.42 148.59 0)
 			(effects
@@
 			)
 		)
-		(property "Footprint" ""
+		(property "Footprint" "Resistor_SMD:R_0805_2012Metric"
 			(at 189.23 109.728 90)
 			(effects
@@
 			)
 		)
-		(property "Footprint" ""
+		(property "Footprint" "Crystal:Crystal_SMD_5032-2Pin_5.0x3.2mm_HandSoldering"
 			(at 34.29 77.47 0)
 			(effects
@@
 			)
 		)
-		(property "Footprint" ""
+		(property "Footprint" "Capacitor_SMD:C_0805_2012Metric"
 			(at 179.07 49.8348 0)
 			(effects
@@
 			)
 		)
-		(property "Footprint" ""
+		(property "Footprint" "Crystal:Crystal_SMD_5032-2Pin_5.0x3.2mm_HandSoldering"
 			(at 187.96 86.36 0)
 			(effects
@@
 			)
 		)
-		(property "Footprint" ""
+		(property "Footprint" "MountingHole:MountingHole_2.1mm"
 			(at 185.42 156.21 0)
 			(effects
@@
 			)
 		)
-		(property "Footprint" ""
+		(property "Footprint" "Package_SO:SOIC-8_5.23x5.23mm_P1.27mm"
 			(at 92.71 165.1 0)
 			(effects
@@
 			)
 		)
-		(property "Footprint" ""
+		(property "Footprint" "Package_SO:SOIC-8_5.23x5.23mm_P1.27mm"
 			(at 59.69 165.1 0)
 			(effects
@@
 			)
 		)
-		(property "Footprint" ""
+		(property "Footprint" "Capacitor_SMD:C_0805_2012Metric"
 			(at 169.8752 83.82 0)
 			(effects
@@
 			)
 		)
-		(property "Footprint" ""
+		(property "Footprint" "LED_SMD:LED_0805_2012Metric"
 			(at 185.42 71.12 0)
 			(effects
@@
 			)
 		)
-		(property "Footprint" ""
+		(property "Footprint" "Capacitor_SMD:C_0805_2012Metric"
 			(at 248.6152 68.58 0)
 			(effects
@@
 			)
 		)
-		(property "Footprint" ""
+		(property "Footprint" "LED_SMD:LED_0805_2012Metric"
 			(at 255.27 87.63 0)
 			(effects
@@
 			)
 		)
-		(property "Footprint" ""
+		(property "Footprint" "Resistor_SMD:R_0805_2012Metric"
 			(at 167.64 72.898 90)
 			(effects
@@
 			)
 		)
-		(property "Footprint" ""
+		(property "Footprint" "Resistor_SMD:R_0805_2012Metric"
 			(at 253.492 99.06 90)
 			(effects
@@
 			)
 		)
-		(property "Footprint" ""
+		(property "Footprint" "Connector_PinHeader_2.54mm:PinHeader_1x02_P2.54mm_Vertical"
 			(at 264.16 61.976 90)
 			(effects
@@
 			)
 		)
-		(property "Footprint" ""
+		(property "Footprint" "MountingHole:MountingHole_2.1mm"
 			(at 185.42 133.35 0)
 			(effects
@@
 			)
 		)
-		(property "Footprint" ""
+		(property "Footprint" "Resistor_SMD:R_0805_2012Metric"
 			(at 123.952 163.83 90)
 			(effects
@@
 			)
 		)
-		(property "Footprint" ""
+		(property "Footprint" "Capacitor_SMD:C_0805_2012Metric"
 			(at 169.8752 96.52 0)
 			(effects
@@
 			)
 		)
-		(property "Footprint" ""
+		(property "Footprint" "Resistor_SMD:R_0805_2012Metric"
 			(at 134.112 163.83 90)
 			(effects
@@
 			)
 		)
-		(property "Footprint" ""
+		(property "Footprint" "Resistor_SMD:R_0805_2012Metric"
 			(at 109.982 74.93 90)
 			(effects
@@
 			)
 		)
-		(property "Footprint" ""
+		(property "Footprint" "Capacitor_SMD:C_0805_2012Metric"
 			(at 127.9652 78.74 0)
 			(effects
@@
 			)
 		)
-		(property "Footprint" ""
+		(property "Footprint" "MountingHole:MountingHole_2.1mm"
 			(at 185.42 140.97 0)
 			(effects
@@
 			)
 		)
-		(property "Footprint" ""
+		(property "Footprint" "Resistor_SMD:R_0805_2012Metric"
 			(at 97.282 74.93 90)
 			(effects

Commit message: added nets to root schematic
Connections:
- net Vcc: now reaches R7.1
- net Vcc: now also C1.1, R1.1, R2.1, R3.1, R6.1, U1.1 (A0), U1.2 (A1), U1.3 (A2), U1.8 (VCC), U2.1 (A0), U2.3 (A2), U2.8 (VCC), U3.8 (VCC)
- net RESET: now reaches R7.2
- net RESET: now also U4.29 (PC6/~{RESET})
- net at Y2.1: now also U3.2 (X2)
- net at Y2.2: now also U3.1 (X1)
- net GND: now reaches C4.1
- net GND: now also BT1.2 (-), C1.2, C2.1, C3.1, C5.2, R4.1, R5.2, U1.4 (GND), U1.7 (WP), U2.2 (A1), U2.4 (GND), U2.7 (WP), U3.4 (GND), U4.21 (GND), U4.3 (GND), U4.5 (GND)
- net at C4.2: now also U4.20 (AREF)
- net D3: now reaches U4.1 (PD3)
- net D6: now reaches U4.10 (PD6)
- net D7: now reaches U4.11 (PD7)
- net D8: now reaches U4.12 (PB0)
- net MOSI: now reaches U4.15 (PB3)
- net MISO: now reaches U4.16 (PB4)
- net SCK: now reaches U4.17 (PB5)
- net SCK: now also D2.2 (A), R6.2, U1.6 (SCL), U2.6 (SCL), U3.6 (SCL), U4.28 (PC5)
- net at U4.18 (AVCC): now also BT1.1 (+), C5.1, D1.2 (A), U4.4 (VCC)
- net D4: now reaches U4.2 (PD4)
- net SDA: now reaches U4.27 (PC4)
- net SDA: now also R1.2, U1.5 (SDA), U2.5 (SDA), U3.5 (SDA)
- net RX: now reaches U4.30 (PD0)
- net TX: now reaches U4.31 (PD1)
- net D2: now reaches U4.32 (PD2)
- net at U4.6 (VCC): no longer U4.4 (VCC)
- net at U4.7 (PB6): now also C3.2, Y1.1
- net at U4.8 (PB7): now also C2.2, Y1.2
- net D5: now reaches U4.9 (PD5)
- net at U3.3 (~{INTA}): now also R3.2
- net at U3.7 (SQW/~INT): now also R2.2
- net at D2.1 (K): now also R4.2
- net at D1.1 (K): now also R5.1
- no-connect marks 0 -> 9
Other:
- moved on the sheet: BT1, C2, C3, C4, C5, D1, D2, R4, R5, R7, U1, Y1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

Commit message: updated nets on both schematics
Other:
- sheet Connectors ports: added D2, D3, D4, D5, D6, D7, D8, GND, MISO, MOSI, RESET, RX, SCK, SDA, TX, Vcc; removed none

Commit message: added comments
Other:
- note added: "EEPROM"
- note added: "MCU"
- note added: "Mounting"
- note added: "Real time clock"
- moved on the sheet: BT1, C1, C2, C3, C4, C5, D1, D2, H1, H2, H3, H4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

Commit message: updated pcb and fixed bat Vcc
Connections:
- net Vcc: now also BT1.1 (+), C5.1, D1.2 (A), U4.18 (AVCC), U4.4 (VCC)
Changed lines of the file:
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@@
+	)
+	(junction
+		(at 110.49 46.99)
+		(diameter 0)
+		(color 0 0 0 0)
 	)
 	(junction
@@
 	(wire
 		(pts
-			(xy 107.95 46.99) (xy 118.11 46.99)
+			(xy 107.95 46.99) (xy 110.49 46.99)
 		)
 		(stroke
@@
 		(pts
 			(xy 24.13 69.85) (xy 24.13 68.58)
+		)
+		(stroke
+			(width 0)
+			(type default)
+		)
+	)
+	(wire
+		(pts
+			(xy 110.49 46.99) (xy 118.11 46.99)
 		)
 		(stroke
@@
 		)
 	)
+	(label "Vcc"
+		(at 266.7 43.18 0)
+		(fields_autoplaced yes)
+		(effects
+			(font
+				(size 1.27 1.27)
+			)
+			(justify left bottom)
+		)
+	)
 	(label "SCK"
 		(at 45.72 57.15 180)
@@
 	(symbol
 		(lib_id "power:PWR_FLAG")
-		(at 107.95 46.99 0)
+		(at 110.49 46.99 0)
 		(unit 1)
 		(exclude_from_sim no)
@@
 		(fields_autoplaced yes)
 		(property "Reference" "#FLG03"
-			(at 107.95 45.085 0)
+			(at 110.49 45.085 0)
 			(effects
 				(font
@@
 		)
 		(property "Value" "PWR_FLAG"
-			(at 107.95 41.91 0)
+			(at 110.49 41.91 0)
 			(effects
 				(font
@@
 		)
 		(property "Footprint" ""
-			(at 107.95 46.99 0)
+			(at 110.49 46.99 0)
 			(effects
 				(font
@@
 		)
 		(property "Datasheet" "~"
-			(at 107.95 46.99 0)
+			(at 110.49 46.99 0)
 			(effects
 				(font
@@
 		)
 		(property "Description" "Special symbol for telling ERC where power comes from"
-			(at 107.95 46.99 0)
+			(at 110.49 46.99 0)
 			(effects
 				(font
