File: mcu-datalogger/mcu-datalogger.kicad_pcb (KiCad board)
At the start: 2 copper layers, 0 parts

Commit message: setup pcb
Parts:
- added BT1: Battery, Connector_PinHeader_2.54mm:PinHeader_1x02_P2.54mm_Vertical, F.Cu at (119.3, 102.4)
- added C1: 0.1uF, Capacitor_SMD:C_0805_2012Metric, F.Cu at (141.6, 92.1)
- added C2: 22pF, Capacitor_SMD:C_0805_2012Metric, F.Cu at (141.6, 95.2)
- added C3: 22pF, Capacitor_SMD:C_0805_2012Metric, F.Cu at (141.6, 98.2)
- added C4: 0.1uF, Capacitor_SMD:C_0805_2012Metric, F.Cu at (141.6, 101.2)
- added C5: 100nF, Capacitor_SMD:C_0805_2012Metric, F.Cu at (141.6, 104.2)
- added D1: LED, LED_SMD:LED_0805_2012Metric, F.Cu at (146.0, 92.2)
- added D2: LED, LED_SMD:LED_0805_2012Metric, F.Cu at (146.0, 95.2)
- added H1: MountingHole, MountingHole:MountingHole_2.1mm, F.Cu at (119.8, 80.0)
- added H2: MountingHole, MountingHole:MountingHole_2.1mm, F.Cu at (119.8, 85.7)
- added H3: MountingHole, MountingHole:MountingHole_2.1mm, F.Cu at (119.8, 91.5)
- added H4: MountingHole, MountingHole:MountingHole_2.1mm, F.Cu at (119.8, 97.2)
- added J1: Conn_01x04_Pin, Connector_PinHeader_2.54mm:PinHeader_1x04_P2.54mm_Vertical, F.Cu at (157.2, 79.4)
- added J2: Conn_01x04_Pin, Connector_PinHeader_2.54mm:PinHeader_1x04_P2.54mm_Vertical, F.Cu at (161.9, 79.4)
- added J3: Conn_01x09_Pin, Connector_PinHeader_2.54mm:PinHeader_1x09_P2.54mm_Vertical, F.Cu at (152.6, 79.4)
- added J4: Conn_02x03_Odd_Even, Connector_PinHeader_2.54mm:PinHeader_2x03_P2.54mm_Vertical, F.Cu at (157.2, 91.7)
- added R1: 4.7k, Resistor_SMD:R_0805_2012Metric, F.Cu at (124.9, 78.6)
- added R2: 10K, Resistor_SMD:R_0805_2012Metric, F.Cu at (124.9, 81.5)
- added R3: 10K, Resistor_SMD:R_0805_2012Metric, F.Cu at (124.9, 84.5)
- added R4: 330, Resistor_SMD:R_0805_2012Metric, F.Cu at (124.9, 87.4)
- added R5: 330, Resistor_SMD:R_0805_2012Metric, F.Cu at (124.9, 90.4)
- added R6: 4.7k, Resistor_SMD:R_0805_2012Metric, F.Cu at (124.9, 93.3)
- added R7: 10K, Resistor_SMD:R_0805_2012Metric, F.Cu at (124.9, 96.3)
- added U1: 24LC1025, Package_SO:SOIC-8_5.23x5.23mm_P1.27mm, F.Cu at (132.3, 80.5)
- added U2: 24LC1025, Package_SO:SOIC-8_5.23x5.23mm_P1.27mm, F.Cu at (132.3, 87.2)
- added U3: DS1337S_, DS1337S_:SOIC127P600X175-8N, F.Cu at (132.3, 105.3)
- added U4: ATMEGA328P-AU, ATMEGA328P-AU:QFP80P900X900X120-32N, F.Cu at (133.7, 96.3)
- added Y1: 16MHz, Crystal:Crystal_SMD_5032-2Pin_5.0x3.2mm_HandSoldering, F.Cu at (142.6, 79.5)
- added Y2: 32.768 KHz, Crystal:Crystal_SMD_5032-2Pin_5.0x3.2mm_HandSoldering, F.Cu at (142.6, 84.4)

Commit message: placed footplrints
Parts:
- moved J3 88.7 mm to (65.1, 94.0), turned to 90 degrees
- moved Y2 81.3 mm to (61.2, 85.2), turned to 90 degrees
- moved J2 72.6 mm to (90.8, 94.0), turned to 90 degrees
- moved C4 70.7 mm to (78.0, 70.0)
- moved U3 65.7 mm to (69.2, 86.8)
- moved C3 65.2 mm to (82.8, 70.0)
- moved U2 64.4 mm to (69.9, 71.4)
- moved C5 64.1 mm to (87.3, 70.0)
- moved BT1 64.0 mm to (61.5, 75.0)
- moved U1 62.9 mm to (69.4, 79.4)
- moved Y1 61.0 mm to (82.2, 88.2)
- moved D2 60.4 mm to (91.8, 68.5)
- moved H1 60.3 mm to (60.5, 69.2)
- moved H4 59.4 mm to (60.5, 94.0)
- moved R2 58.4 mm to (67.3, 91.2)
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
Commit message: routed pcb
Parts:
- moved C4 24.4 mm to (92.0, 90.0), turned to 180 degrees
- moved C1 23.7 mm to (78.5, 69.5)
- moved R6 4.75 mm to (91.9, 81.8)
- moved H1 3.89 mm to (57.8, 66.5)
- moved H4 3.72 mm to (57.8, 96.5)
- moved H2 3.54 mm to (107.0, 66.5)
- moved H3 3.54 mm to (107.0, 96.5)
- moved R1 3.01 mm to (91.8, 78.0)
- moved Y2 1.25 mm to (61.2, 86.5)
- moved BT1 1.03 mm to (61.2, 76.0)
- moved D1 1.03 mm to (96.6, 69.5)
- moved D2 1.03 mm to (92.1, 69.5)
- moved R4 1.00 mm to (92.1, 74.0)
- moved R5 1.00 mm to (96.3, 74.0), turned to 0 degrees
- moved R7 1.00 mm to (96.3, 78.0)
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Routing:
- net GND: track 0.00 -> 180.9 mm, vias 0 -> 20
- net /Vcc: track 0.00 -> 145.8 mm, vias 0 -> 8
- net /SCK: track 0.00 -> 104.8 mm, vias 0 -> 17
- net /SDA: track 0.00 -> 89.1 mm, vias 0 -> 2
- net Net-(BT1-+): track 0.00 -> 67.5 mm, vias 0 -> 8
- net /MOSI: track 0.00 -> 29.0 mm
- net /TX: track 0.00 -> 28.6 mm, vias 0 -> 2
- net /MISO: track 0.00 -> 28.3 mm
- net /D2: track 0.00 -> 27.9 mm, vias 0 -> 2
- net /RX: track 0.00 -> 25.6 mm, vias 0 -> 2
- net Net-(U4-PB6): track 0.00 -> 24.7 mm
- net /RESET: track 0.00 -> 23.6 mm, vias 0 -> 2
- net /D3: track 0.00 -> 22.5 mm, vias 0 -> 2
- net /D4: track 0.00 -> 20.9 mm, vias 0 -> 2
- net Net-(U4-PB7): track 0.00 -> 19.3 mm
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- added copper zone on F.Cu, net /Vcc
- added copper zone on B.Cu, net GND
Other:
- board outline added: 55.2 x 36 mm

Commit message: routing complete
Routing:
- net Net-(BT1-+): track 67.5 -> 77.2 mm
- net /SCK: track 104.8 -> 107.4 mm, vias 17 -> 14
- net Net-(U4-AREF): track 13.9 -> 14.5 mm
- net GND: track 180.9 -> 180.7 mm, vias 20 -> 18

Commit message: updated pcb and fixed bat Vcc
Connections:
- BT1 pad 1: Net-(BT1-+) -> /Vcc
- C5 pad 1: Net-(BT1-+) -> /Vcc
- D1 pad 2: Net-(BT1-+) -> /Vcc
- U4 pad 18: Net-(BT1-+) -> /Vcc
- U4 pad 4: Net-(BT1-+) -> /Vcc
Routing:
- net Net-(BT1-+): track 77.2 -> 0.00 mm, vias 8 -> 0
- net /Vcc: track 145.8 -> 218.9 mm, vias 8 -> 16
- removed copper zone on F.Cu, net /Vcc
Other:
- board text added: "Vcc"

Commit message: finished 2-layer pcb
Other:
- board text added: "0.0000 mm / 0.0000 mm"
- board text added: "0.3000 mm"
- board text added: "1.6000 mm"
- board text added: "2"
- board text added: "55.2540 mm x 36.0040 mm"
- board text added: "BOARD CHARACTERISTICS"
- board text added: "Board Thickness:"
- board text added: "Board overall dimensions:"
- board text added: "Castellated pads:"
- board text added: "Copper Finish:"
- board text added: "Copper Layer Count:"
- board text added: "Edge card connectors:"
- board text added: "Impedance Control:"
- board text added: "Min hole diameter:"
- board text added: "Min track/spacing:"
- board text added: "No"
- board text added: "None"
- board text added: "Plated Board Edge:"
